File: _autosave-kr_1.sch (KiCad schematic (older format))
At the start: 14 parts

Commit message: switchs
Parts:
- added F?: 500mA, symbol Device:Polyfuse_Small
- added MX? (x14): MX-NoLED, symbol MX_Alps_Hybrid:MX-NoLED
- added USB?: Molex-0548190589, symbol random-keyboard-parts:Molex-0548190589
Connections:
- net +5V: now also F?.2
- net D+: now also USB?.3 (D+)
- net D-: now also USB?.4 (D-)
- net GND: now also USB?.1 (GND)
- new net VCC: F?.1, USB?.5 (VBUS)
Other:
- moved on the sheet: C?, R?, SW?, U?, Y?
